Commit message: Fixed collision checking

File: franka_ros/franka_description/robots/panda/panda.urdf.xacro (robot description, xacro)
@@ -43,4 +43,54 @@
       </geometry>
     </visual>
+    <collision>
+      <geometry>
+        <box size="0.0078 0.130 0.0192"/>
+      </geometry>
+      <surface>
+          <friction>
+            <ode>
+              <mu>1</mu>
+              <mu2>1</mu2>
+              <fdir1>0 0 0</fdir1>
+              <slip1>0</slip1>
+              <slip2>0</slip2>
+            </ode>
+            <torsional>
+              <coefficient>1</coefficient>
+              <patch_radius>0</patch_radius>
+              <surface_radius>0</surface_radius>
+              <use_patch_radius>1</use_patch_radius>
+              <ode>
+                <slip>0</slip>
+              </ode>
+            </torsional>
+          </friction>
+          <bounce>
+            <restitution_coefficient>0</restitution_coefficient>
+            <threshold>1e+06</threshold>
+          </bounce>
+          <contact>
+            <collide_without_contact>0</collide_without_contact>
+            <collide_without_contact_bitmask>1</collide_without_contact_bitmask>
+            <collide_bitmask>1</collide_bitmask>
+            <ode>
+              <soft_cfm>0</soft_cfm>
+              <soft_erp>0.2</soft_erp>
+              <kp>1e+13</kp>
+              <kd>1</kd>
+              <max_vel>0.01</max_vel>
+              <min_depth>0</min_depth>
+            </ode>
+            <bullet>
+              <split_impulse>1</split_impulse>
+              <split_impulse_penetration_threshold>-0.01</split_impulse_penetration_threshold>
+              <soft_cfm>0</soft_cfm>
+              <soft_erp>0.2</soft_erp>
+              <kp>1e+13</kp>
+              <kd>1</kd>
+            </bullet>
+          </contact>
+        </surface>
+    </collision>
   </link>
   <joint name="camera_optical_joint" type="fixed">

Commit message: Updated dope detector code

File: franka_ros/franka_description/robots/panda/panda.urdf.xacro (robot description, xacro)
@@ -95,5 +95,5 @@
   </link>
   <joint name="camera_optical_joint" type="fixed">
-    <origin xyz="0 0 0" rpy="${-pi/2} 0 ${-pi/2}" />
+    <origin xyz="0 0 0" rpy="${0} ${pi} ${0}" />
     <parent link="camera_link" />
     <child link="camera_link_optical" />
